Commit message: Redesign printed joints for owned heat-set inserts

File: sim/beni.urdf (robot description, URDF)
Before this commit: robot beni_prototype1, 7 links, 6 joints
Links:
- link base_link: mass 1.613706 -> 1.628720
- link l_shank: mass 0.409285 -> 0.410591
- link l_thigh: mass 0.219845 -> 0.222429
- link l_wheel: mass 0.209090 -> 0.207060
- link r_shank: mass 0.409285 -> 0.410591
- link r_thigh: mass 0.219845 -> 0.222429
- link r_wheel: mass 0.209090 -> 0.207060
